Commit message: lidar-only mapping with some small mod on model/control

File: urdf/agv_2wheels.urdf (robot description, URDF)
Before this commit: robot agv_2wheels, 7 links, 6 joints
Links:
- link chassis: mass 15.0 -> 5.0
- link left_wheel: mass 5.0 -> 1.0
- link right_wheel: mass 5.0 -> 1.0

File: urdf/agv_2wheels.xacro (robot description, xacro)
@@ -11,5 +11,5 @@
     <pose>0 0 0.1 0 0 0</pose>
     <inertial>
-      <mass value="15.0" />
+      <mass value="5.0" />
       <origin xyz="0.0 0 0" rpy=" 0 0 0" />
       <inertia
@@ -79,5 +79,5 @@
   <link name="left_wheel">
     <inertial>
-      <mass value="5.0" />
+      <mass value="1.0" />
       <origin xyz="0 0 0" rpy=" 0 1.5707 1.5707" />
       <inertia
@@ -112,5 +112,5 @@
   <link name="right_wheel">
     <inertial>
-      <mass value="5.0" />
+      <mass value="1.0" />
       <origin xyz="0 0 0" rpy="0 1.5707 1.5707" />
       <inertia
